File: entradas_digitales.sch (KiCad schematic (older format))
At the start: 68 parts, among them J1 Opto5-8, J2 Opto1-4, J3 Entrada, J4 Salida, U1 TLP627-4, U2 TLP627-4, U3 4021

Commit message: Agregado de BOM
Parts:
- D1, D10, D11, D12, D13, D14, D15, D16, D17, D27: value LED -> 17-21SURC/S530-A3/TR8
- D18, D19, D20, D21, D22, D23, D24, D25, D26: value LED -> 17-21SYGC/S530-E2/TR8
- D2: value KDZVTFTR12B -> MMSZ5242BTR
- D3, D4, D5, D6, D7, D8, D9: value D_Zener -> MMSZ5242BTR
- R1, R10, R11, R12, R13, R14, R15, R16, R17, R2, R27, R28, R3, R4, R5, R6, R7, R8, R9: value R -> 10K
- R18, R19, R20, R21, R22, R23, R24, R25, R26: value R -> 2K2
- U1, U2: value TLP627-4 -> LTV-845
Connections:
- net 24V-A: no longer R2.1, R3.1, R4.1, R5.1
- net 24V-B: no longer R6.1, R7.1, R8.1, R9.1
- net at D2.2 (A), R10.2: now also R2.1
- net at D3.2 (A), R11.2: now also R3.1
- net at D4.2 (A), R12.2: now also R4.1
- net at D5.2 (A), R13.2: now also R5.1
- net at D6.2 (A), R14.2: now also R6.1
- net at D7.2 (A), R15.2: now also R7.1
- net at D8.2 (A), R16.2: now also R8.1
- net at D9.2 (A), R17.2: now also R9.1
